Commit message: feat (UNTESTED): add node to correct LIDAR position on car

File: src/car_description/urdf/car.urdf.xacro (robot description, xacro)
@@ -1,10 +1,11 @@
-bot xmlns:xacro="http://www.ros.org/wiki/xacro" name="car">
+<?xml version="1.0"?>
+<robot xmlns:xacro="http://www.ros.org/wiki/xacro" name="car">
   <!-- Base -->
   <link name="base_link"/>
   <!-- LiDAR -->
-  <link name="laser"/>
-  <joint name="laser_joint" type="fixed">
+  <link name="scan"/>
+  <joint name="scan_joint" type="fixed">
     <parent link="base_link"/>
-    <child link="laser"/>
+    <child link="scan"/>
     <origin xyz="-0.5 0.0 0.25" rpy="0 0 0"/>
   </joint>
